File: hardware/DATA_LOGER_IOT.kicad_pcb (KiCad board)
At the start: 2 copper layers, 0 parts

Commit message: WIP: guardar cambios antes de pull
Parts:
- added REF** (x6): ESP32-S3-WROOM-1, ESP32-S3-WROOM-1, F.Cu at (35.0, 22.0)
- added REF**: JST_PH_B2B-PH-K_1x02_P2.00mm_Vertical, JST_PH_B2B-PH-K_1x02_P2.00mm_Vertical, F.Cu at (15.0, 48.0)
- added REF** (x2): TI_SO-PowerPAD-8, TI_SO-PowerPAD-8, F.Cu at (35.0, 48.0)
Routing:
- net +12V: track 0.00 -> 20.0 mm
- added copper zone on B.Cu, net GND
- added copper zone on F.Cu, net GND
Other:
- board outline added: 50 x 50 mm
- net class Power added: clearance 4.0, trace_width 0.5

Commit message: WIP: guardar cambios antes de pull
Parts:
- removed REF** (x5): ESP32-S3-WROOM-1, ESP32-S3-WROOM-1
- removed REF**: TI_SO-PowerPAD-8, TI_SO-PowerPAD-8
- J1: renamed from REF**; value JST_PH_B2B-PH-K_1x02_P2.00mm_Vertical -> (none)
- U1: renamed from REF**; value ESP32-S3-WROOM-1 -> ESP32-S3
- U2: renamed from REF**; value TI_SO-PowerPAD-8 -> (none)
Connections:
- J1 pad 1: (no net) -> +12V
- J1 pad 2: (no net) -> GND
- U2 pad 7: (no net) -> +12V
- U2 pad 9: (no net) -> GND
Routing:
- net (no net): track 42.4 -> 0.00 mm
Other:
- outline, holes or cut-outs redrawn
- net class Power removed
